File: kicad/v0.0/_autosave-v0.0.kicad_pcb (KiCad board)
At the start: 2 copper layers, 62 parts, among them J1 USB_B_Micro, J2 9V_IN, J3 LED, J4 MOTOR, J5 LED, J6 MOTOR, Q1 IRF520, Q2 IRF520, SW1 SW_Push, SW2 SW_Push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

Commit message: ready to design PCB
Routing:
- net /3V3: track 34.5 -> 0.55 mm
Changed lines of the file:
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@@
   (segment (start 250.3 113.3) (end 236.85 113.3) (width 0.25) (layer "F.Cu") (net 11))
   (segment (start 236.85 113.3) (end 236.525 112.975) (width 0.25) (layer "F.Cu") (net 11))
-  (segment (start 228.225 95.25) (end 240.575 82.9) (width 0.25) (layer "F.Cu") (net 13))
   (segment (start 240.575 82.9) (end 240.575 82.35) (width 0.25) (layer "F.Cu") (net 13))
-  (segment (start 228.225 95.25) (end 230.615 95.25) (width 0.25) (layer "F.Cu") (net 13))
-  (segment (start 230.615 95.25) (end 240.575 105.21) (width 0.25) (layer "F.Cu") (net 13))
   (zone (net 3) (net_name "GND") (layers F&B.Cu) (hatch edge 0.508)
     (connect_pads (clearance 0.508))
