File: kicad/v0.0/v0.0.kicad_sch (KiCad schematic)
At the start: 53 parts, among them J1 USB_B_Micro, J2 9V_IN, J3 LED, J4 MOTOR, Q1 IRF520, SW1 RST, SW2 FLASH, SW3 OPEN/CLOSE, U1 MCP2221AxSL, U2 MAX14872ETC+, U3 ESP32-WROOM-32, U6 AZ1117-3.3

Commit message: blah
Other:
- moved on the sheet: TP10, TP11, TP12, TP8
Changed lines of the file:
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@@
     (pin "1")
   )
-  (symbol (lib_id "Connector:TestPoint") (at 168.91 48.26 0) (unit 1)
-    (in_bom yes) (on_board yes) (fields_autoplaced)
-    (property "Reference" "TP12" (id 0) (at 171.45 43.6879 0)
-      (effects (font (size 1.27 1.27)) (justify left))
-    )
-    (property "Value" "TestPoint" (id 1) (at 171.45 46.2279 0)
-      (effects (font (size 1.27 1.27)) (justify left))
-    )
-    (property "Footprint" "TestPoint:TestPoint_Pad_2.5x2.5mm" (id 2) (at 173.99 48.26 0)
-      (effects (font (size 1.27 1.27)) hide)
-    )
-    (property "Datasheet" "~" (id 3) (at 173.99 48.26 0)
+  (symbol (lib_id "Connector:TestPoint") (at 166.37 38.1 0) (unit 1)
+    (in_bom yes) (on_board yes) (fields_autoplaced)
+    (property "Reference" "TP12" (id 0) (at 168.91 33.5279 0)
+      (effects (font (size 1.27 1.27)) (justify left))
+    )
+    (property "Value" "TestPoint" (id 1) (at 168.91 36.0679 0)
+      (effects (font (size 1.27 1.27)) (justify left))
+    )
+    (property "Footprint" "TestPoint:TestPoint_Pad_2.5x2.5mm" (id 2) (at 171.45 38.1 0)
+      (effects (font (size 1.27 1.27)) hide)
+    )
+    (property "Datasheet" "~" (id 3) (at 171.45 38.1 0)
       (effects (font (size 1.27 1.27)) hide)
     )
@@
     (pin "2")
   )
-  (symbol (lib_id "Connector:TestPoint") (at 168.91 38.1 0) (unit 1)
-    (in_bom yes) (on_board yes) (fields_autoplaced)
-    (property "Reference" "TP11" (id 0) (at 171.45 33.5279 0)
-      (effects (font (size 1.27 1.27)) (justify left))
-    )
-    (property "Value" "TestPoint" (id 1) (at 171.45 36.0679 0)
-      (effects (font (size 1.27 1.27)) (justify left))
-    )
-    (property "Footprint" "TestPoint:TestPoint_Pad_2.5x2.5mm" (id 2) (at 173.99 38.1 0)
-      (effects (font (size 1.27 1.27)) hide)
-    )
-    (property "Datasheet" "~" (id 3) (at 173.99 38.1 0)
+  (symbol (lib_id "Connector:TestPoint") (at 151.765 38.1 0) (unit 1)
+    (in_bom yes) (on_board yes) (fields_autoplaced)
+    (property "Reference" "TP11" (id 0) (at 154.305 33.5279 0)
+      (effects (font (size 1.27 1.27)) (justify left))
+    )
+    (property "Value" "TestPoint" (id 1) (at 154.305 36.0679 0)
+      (effects (font (size 1.27 1.27)) (justify left))
+    )
+    (property "Footprint" "TestPoint:TestPoint_Pad_2.5x2.5mm" (id 2) (at 156.845 38.1 0)
+      (effects (font (size 1.27 1.27)) hide)
+    )
+    (property "Datasheet" "~" (id 3) (at 156.845 38.1 0)
       (effects (font (size 1.27 1.27)) hide)
     )
@@
     (pin "2")
   )
-  (symbol (lib_id "Connector:TestPoint") (at 153.67 48.26 0) (unit 1)
-    (in_bom yes) (on_board yes) (fields_autoplaced)
-    (property "Reference" "TP8" (id 0) (at 156.21 43.6879 0)
-      (effects (font (size 1.27 1.27)) (justify left))
-    )
-    (property "Value" "TestPoint" (id 1) (at 156.21 46.2279 0)
-      (effects (font (size 1.27 1.27)) (justify left))
-    )
-    (property "Footprint" "TestPoint:TestPoint_Pad_2.5x2.5mm" (id 2) (at 158.75 48.26 0)
-      (effects (font (size 1.27 1.27)) hide)
-    )
-    (property "Datasheet" "~" (id 3) (at 158.75 48.26 0)
+  (symbol (lib_id "Connector:TestPoint") (at 108.585 37.465 0) (unit 1)
+    (in_bom yes) (on_board yes) (fields_autoplaced)
+    (property "Reference" "TP8" (id 0) (at 111.125 32.8929 0)
+      (effects (font (size 1.27 1.27)) (justify left))
+    )
+    (property "Value" "TestPoint" (id 1) (at 111.125 35.4329 0)
+      (effects (font (size 1.27 1.27)) (justify left))
+    )
+    (property "Footprint" "TestPoint:TestPoint_Pad_2.5x2.5mm" (id 2) (at 113.665 37.465 0)
+      (effects (font (size 1.27 1.27)) hide)
+    )
+    (property "Datasheet" "~" (id 3) (at 113.665 37.465 0)
       (effects (font (size 1.27 1.27)) hide)
     )
@@
     (pin "1")
   )
-  (symbol (lib_id "Connector:TestPoint") (at 122.555 47.625 0) (unit 1)
-    (in_bom yes) (on_board yes) (fields_autoplaced)
-    (property "Reference" "TP10" (id 0) (at 125.095 43.0529 0)
-      (effects (font (size 1.27 1.27)) (justify left))
-    )
-    (property "Value" "TestPoint" (id 1) (at 125.095 45.5929 0)
-      (effects (font (size 1.27 1.27)) (justify left))
-    )
-    (property "Footprint" "TestPoint:TestPoint_Pad_2.5x2.5mm" (id 2) (at 127.635 47.625 0)
-      (effects (font (size 1.27 1.27)) hide)
-    )
-    (property "Datasheet" "~" (id 3) (at 127.635 47.625 0)
-      (effects (font (size 1.27 1.27)) hide)
-    )
+  (symbol (lib_id "Connector:TestPoint") (at 137.16 38.1 0) (unit 1)
+    (in_bom yes) (on_board yes) (fields_autoplaced)
+    (property "Reference" "TP10" (id 0) (at 139.7 33.5279 0)
+      (effects (font (size 1.27 1.27)) (justify left))
+    )
+    (property "Value" "TestPoint" (id 1) (at 139.7 36.0679 0)
+      (effects (font (size 1.27 1.27)) (justify left))
+    )
+    (property "Footprint" "TestPoint:TestPoint_Pad_2.5x2.5mm" (id 2) (at 142.24 38.1 0)
+      (effects (font (size 1.27 1.27)) hide)
+    )
+    (property "Datasheet" "~" (id 3) (at 142.24 38.1 0)
+      (effects (font (size 1.27 1.27)) hide)
+    )

Commit message: mbro isnt being such a bro
Parts:
- removed D1, D2: D, Diode_SMD:D_SMA_Handsoldering, symbol Device:D
- added D1, D2: MBR0520, Diode_SMD:D_SOD-123, symbol Diode:MBR0520
Connections:
- net +3V3: now also D1.1 (K), D2.1 (K)
- net at C10.1, TP5.1, U6.2 (VO): now also D2.2 (A)
- net at C3.1, TP6.1, U1.11 (VUSB): now also D1.2 (A)
Changed lines of the file:
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@@
     (pin "1")
+  )
+  (symbol (lib_id "Diode:MBR0520") (at 69.85 143.51 180) (unit 1)
+    (in_bom yes) (on_board yes) (fields_autoplaced)
+    (property "Reference" "D1" (id 0) (at 70.1675 137.16 0))
+    (property "Value" "MBR0520" (id 1) (at 70.1675 139.7 0))
+    (property "Footprint" "Diode_SMD:D_SOD-123" (id 2) (at 69.85 139.065 0)
+      (effects (font (size 1.27 1.27)) hide)
+    )
+    (property "Datasheet" "http://www.mccsemi.com/up_pdf/MBR0520~MBR0580(SOD123).pdf" (id 3) (at 69.85 143.51 0)
+      (effects (font (size 1.27 1.27)) hide)
+    )
+    (pin "1")
+    (pin "2")
   )
   (symbol (lib_id "Connector:TestPoint") (at 166.37 38.1 0) (unit 1)
@@
     (pin "1")
   )
-  (symbol (lib_id "Device:D") (at 262.89 33.655 180) (unit 1)
-    (in_bom yes) (on_board yes) (fields_autoplaced)
-    (property "Reference" "D1" (id 0) (at 262.89 26.67 0))
-    (property "Value" "D" (id 1) (at 262.89 29.21 0))
-    (property "Footprint" "Diode_SMD:D_SMA_Handsoldering" (id 2) (at 262.89 33.655 0)
-      (effects (font (size 1.27 1.27)) hide)
-    )
-    (property "Datasheet" "~" (id 3) (at 262.89 33.655 0)
-      (effects (font (size 1.27 1.27)) hide)
-    )
-    (pin "1")
-    (pin "2")
-  )
   (symbol (lib_id "Device:C") (at 40.005 76.2 0) (unit 1)
     (in_bom yes) (on_board yes) (fields_autoplaced)
@@
     (pin "1")
   )
-  (symbol (lib_id "Device:D") (at 69.85 143.51 180) (unit 1)
-    (in_bom yes) (on_board yes) (fields_autoplaced)
-    (property "Reference" "D2" (id 0) (at 69.85 137.16 0))
-    (property "Value" "D" (id 1) (at 69.85 139.7 0))
-    (property "Footprint" "Diode_SMD:D_SMA_Handsoldering" (id 2) (at 69.85 143.51 0)
-      (effects (font (size 1.27 1.27)) hide)
-    )
-    (property "Datasheet" "~" (id 3) (at 69.85 143.51 0)
-      (effects (font (size 1.27 1.27)) hide)
-    )
-    (pin "1")
-    (pin "2")
-  )
   (symbol (lib_id "Device:R") (at 53.34 30.48 90) (unit 1)
     (in_bom yes) (on_board yes) (fields_autoplaced)
@@
     )
     (property "Datasheet" "~" (id 3) (at 45.72 36.83 0)
+      (effects (font (size 1.27 1.27)) hide)
+    )
+    (pin "1")
+    (pin "2")
+  )
+  (symbol (lib_id "Diode:MBR0520") (at 262.89 33.655 180) (unit 1)
+    (in_bom yes) (on_board yes) (fields_autoplaced)
+    (property "Reference" "D2" (id 0) (at 263.2075 26.67 0))
+    (property "Value" "MBR0520" (id 1) (at 263.2075 29.21 0))
+    (property "Footprint" "Diode_SMD:D_SOD-123" (id 2) (at 262.89 29.21 0)
+      (effects (font (size 1.27 1.27)) hide)
+    )
+    (property "Datasheet" "http://www.mccsemi.com/up_pdf/MBR0520~MBR0580(SOD123).pdf" (id 3) (at 262.89 33.655 0)
       (effects (font (size 1.27 1.27)) hide)
     )
@@
       (reference "C14") (unit 1) (value "470u") (footprint "Capacitor_THT:CP_Radial_D10.0mm_P5.00mm")
     )
-    (path "/3d4457ec-30ce-45fc-a96c-68de8677bea1"
-      (reference "D1") (unit 1) (value "D") (footprint "Diode_SMD:D_SMA_Handsoldering")
-    )
-    (path "/e3a0fe9d-5724-4b53-8844-5d59e367b59e"
-      (reference "D2") (unit 1) (value "D") (footprint "Diode_SMD:D_SMA_Handsoldering")
+    (path "/0382b9c4-ee92-4a09-8b03-d2428df3f286"
+      (reference "D1") (unit 1) (value "MBR0520") (footprint "Diode_SMD:D_SOD-123")
+    )
+    (path "/f5fe6829-1c88-450d-ae62-8c35262f0e11"
+      (reference "D2") (unit 1) (value "MBR0520") (footprint "Diode_SMD:D_SOD-123")
     )
     (path "/487c7076-3ee5-4402-975b-6c5bdb52c6fd"

Commit message: general layout ready to be finalized
Parts:
- removed J3: LED, Connector_Molex:Molex_KK-254_AE-6410-02A_1x02_P2.54mm_Vertical, symbol Connector:Conn_01x02_Female
- removed J4: MOTOR, Connector_Molex:Molex_KK-254_AE-6410-02A_1x02_P2.54mm_Vertical, symbol Connector:Conn_01x02_Female
- removed SW3: OPEN/CLOSE, Button_Switch_THT:SW_PUSH-12mm, symbol Switch:SW_Push
- added J3: MOTOR, Connector_Molex:Molex_KK-254_AE-6410-02A_1x02_P2.54mm_Vertical, symbol Connector:Conn_01x02_Male
- added J4: LED, Connector_Molex:Molex_KK-254_AE-6410-04A_1x04_P2.54mm_Vertical, symbol Connector:Conn_01x04_Male
- added J5: BUTTON, Connector_Molex:Molex_KK-254_AE-6410-02A_1x02_P2.54mm_Vertical, symbol Connector:Conn_01x02_Male
Connections:
- net +3V3: now also J5.2 (Pin_2)
- net GND: now also J4.1 (Pin_1)
- net at U2.11 (M2): now also J3.1 (Pin_1)
- net at U2.2 (M1): now also J3.2 (Pin_2)
- net at R3.1, R4.1, TP7.1: now also J5.1 (Pin_1)
- net at R5.2: now also J4.2 (Pin_2), J4.3 (Pin_3), J4.4 (Pin_4)
