File: kicad/v0.0/v0.0.kicad_sch (KiCad schematic)
At the start: 53 parts, among them J1 USB_B_Micro, J2 9V_IN, J3 MOTOR, J4 LED, J5 BUTTON, Q1 IRF520, SW1 RST, SW2 FLASH, U1 MCP2221AxSL, U2 MAX14872ETC+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

Commit message: ready for board review/ordering
Parts:
- removed TP10, TP11, TP12: TestPoint, TestPoint:TestPoint_Pad_2.5x2.5mm, symbol Connector:TestPoint
- SW1: value RST -> RESET
Connections:
- net at TP8.1: now also U3.11 (IO26)
- net at TP9.1: now also U3.37 (IO23)
Other:
- moved on the sheet: TP8, TP9
Changed lines of the file:
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@@
+    (stroke (width 0) (type default) (color 0 0 0 0))
+  )
+  (wire (pts (xy 172.085 130.175) (xy 175.26 130.175))
     (stroke (width 0) (type default) (color 0 0 0 0))
   )
@@
   )
   (wire (pts (xy 45.72 30.48) (xy 45.72 33.02))
+    (stroke (width 0) (type default) (color 0 0 0 0))
+  )
+  (wire (pts (xy 172.085 135.255) (xy 179.07 135.255))
     (stroke (width 0) (type default) (color 0 0 0 0))
   )
@@
     (pin "1")
     (pin "2")
-  )
-  (symbol (lib_id "Connector:TestPoint") (at 166.37 38.1 0) (unit 1)
-    (in_bom yes) (on_board yes) (fields_autoplaced)
-    (property "Reference" "TP12" (id 0) (at 168.91 33.5279 0)
-      (effects (font (size 1.27 1.27)) (justify left))
-    )
-    (property "Value" "TestPoint" (id 1) (at 168.91 36.0679 0)
-      (effects (font (size 1.27 1.27)) (justify left))
-    )
-    (property "Footprint" "TestPoint:TestPoint_Pad_2.5x2.5mm" (id 2) (at 171.45 38.1 0)
-      (effects (font (size 1.27 1.27)) hide)
-    )
-    (property "Datasheet" "~" (id 3) (at 171.45 38.1 0)
-      (effects (font (size 1.27 1.27)) hide)
-    )
-    (pin "1")
   )
   (symbol (lib_id "power:GND") (at 242.57 46.355 0) (unit 1)
@@
       (effects (font (size 1.27 1.27)) (justify left))
     )
-    (property "Value" "RST" (id 1) (at 121.539 97.79 0))
+    (property "Value" "RESET" (id 1) (at 121.539 97.79 0))
     (property "Footprint" "Button_Switch_THT:SW_PUSH-12mm_Wuerth-430476085716" (id 2) (at 114.935 97.79 0)
       (effects (font (size 1.27 1.27)) hide)
@@
     (pin "1")
     (pin "2")
-  )
-  (symbol (lib_id "Connector:TestPoint") (at 151.765 38.1 0) (unit 1)
-    (in_bom yes) (on_board yes) (fields_autoplaced)
-    (property "Reference" "TP11" (id 0) (at 154.305 33.5279 0)
-      (effects (font (size 1.27 1.27)) (justify left))
-    )
-    (property "Value" "TestPoint" (id 1) (at 154.305 36.0679 0)
-      (effects (font (size 1.27 1.27)) (justify left))
-    )
-    (property "Footprint" "TestPoint:TestPoint_Pad_2.5x2.5mm" (id 2) (at 156.845 38.1 0)
-      (effects (font (size 1.27 1.27)) hide)
-    )
-    (property "Datasheet" "~" (id 3) (at 156.845 38.1 0)
-      (effects (font (size 1.27 1.27)) hide)
-    )
-    (pin "1")
   )
   (symbol (lib_id "Mechanical:MountingHole") (at 164.465 26.035 0) (unit 1)
@@
     (pin "2")
   )
-  (symbol (lib_id "Connector:TestPoint") (at 108.585 37.465 0) (unit 1)
-    (in_bom yes) (on_board yes) (fields_autoplaced)
-    (property "Reference" "TP8" (id 0) (at 111.125 32.8929 0)
-      (effects (font (size 1.27 1.27)) (justify left))
-    )
-    (property "Value" "TestPoint" (id 1) (at 111.125 35.4329 0)
-      (effects (font (size 1.27 1.27)) (justify left))
-    )
-    (property "Footprint" "TestPoint:TestPoint_Pad_2.5x2.5mm" (id 2) (at 113.665 37.465 0)
-      (effects (font (size 1.27 1.27)) hide)
-    )
-    (property "Datasheet" "~" (id 3) (at 113.665 37.465 0)
+  (symbol (lib_id "Connector:TestPoint") (at 179.07 135.255 0) (unit 1)
+    (in_bom yes) (on_board yes) (fields_autoplaced)
+    (property "Reference" "TP8" (id 0) (at 181.61 130.6829 0)
+      (effects (font (size 1.27 1.27)) (justify left))
+    )
+    (property "Value" "TestPoint" (id 1) (at 181.61 133.2229 0)
+      (effects (font (size 1.27 1.27)) (justify left))
+    )
+    (property "Footprint" "TestPoint:TestPoint_Pad_2.5x2.5mm" (id 2) (at 184.15 135.255 0)
+      (effects (font (size 1.27 1.27)) hide)
+    )
+    (property "Datasheet" "~" (id 3) (at 184.15 135.255 0)
       (effects (font (size 1.27 1.27)) hide)
     )
@@
     (pin "1")
   )
-  (symbol (lib_id "Connector:TestPoint") (at 122.555 38.1 0) (unit 1)
-    (in_bom yes) (on_board yes) (fields_autoplaced)
-    (property "Reference" "TP9" (id 0) (at 125.095 33.5279 0)
-      (effects (font (size 1.27 1.27)) (justify left))
-    )
-    (property "Value" "TestPoint" (id 1) (at 125.095 36.0679 0)
-      (effects (font (size 1.27 1.27)) (justify left))
-    )
-    (property "Footprint" "TestPoint:TestPoint_Pad_2.5x2.5mm" (id 2) (at 127.635 38.1 0)
-      (effects (font (size 1.27 1.27)) hide)
-    )
-    (property "Datasheet" "~" (id 3) (at 127.635 38.1 0)
+  (symbol (lib_id "Connector:TestPoint") (at 175.26 130.175 0) (unit 1)
+    (in_bom yes) (on_board yes) (fields_autoplaced)
+    (property "Reference" "TP9" (id 0) (at 177.8 125.6029 0)
+      (effects (font (size 1.27 1.27)) (justify left))
+    )
+    (property "Value" "TestPoint" (id 1) (at 177.8 128.1429 0)
+      (effects (font (size 1.27 1.27)) (justify left))
+    )
+    (property "Footprint" "TestPoint:TestPoint_Pad_2.5x2.5mm" (id 2) (at 180.34 130.175 0)
+      (effects (font (size 1.27 1.27)) hide)
+    )
+    (property "Datasheet" "~" (id 3) (at 180.34 130.175 0)
       (effects (font (size 1.27 1.27)) hide)
     )
@@
     )
     (property "Datasheet" "~" (id 3) (at 191.77 114.935 0)
-      (effects (font (size 1.27 1.27)) hide)
-    )
-    (pin "1")
-  )
-  (symbol (lib_id "Connector:TestPoint") (at 137.16 38.1 0) (unit 1)
-    (in_bom yes) (on_board yes) (fields_autoplaced)
-    (property "Reference" "TP10" (id 0) (at 139.7 33.5279 0)
-      (effects (font (size 1.27 1.27)) (justify left))
-    )
-    (property "Value" "TestPoint" (id 1) (at 139.7 36.0679 0)
-      (effects (font (size 1.27 1.27)) (justify left))
-    )
-    (property "Footprint" "TestPoint:TestPoint_Pad_2.5x2.5mm" (id 2) (at 142.24 38.1 0)
-      (effects (font (size 1.27 1.27)) hide)
-    )
-    (property "Datasheet" "~" (id 3) (at 142.24 38.1 0)
       (effects (font (size 1.27 1.27)) hide)
     )
@@
     )
     (path "/53d21e73-5bfa-4153-b844-8c5b7eee3599"
-      (reference "SW1") (unit 1) (value "RST") (footprint "Button_Switch_THT:SW_PUSH-12mm_Wuerth-430476085716")
+      (reference "SW1") (unit 1) (value "RESET") (footprint "Button_Switch_THT:SW_PUSH-12mm_Wuerth-430476085716")
     )
     (path "/1104a2fc-60d0-4d59-8b7e-45420f9c2fda"
@@
       (reference "TP9") (unit 1) (value "TestPoint") (footprint "TestPoint:TestPoint_Pad_2.5x2.5mm")
     )
-    (path "/de818e6e-a56c-46de-b1ed-265dc9caf995"
-      (reference "TP10") (unit 1) (value "TestPoint") (footprint "TestPoint:TestPoint_Pad_2.5x2.5mm")
-    )
-    (path "/69686af5-c79b-4d03-be66-2e9cc08b96ae"
-      (reference "TP11") (unit 1) (value "TestPoint") (footprint "TestPoint:TestPoint_Pad_2.5x2.5mm")
-    )
-    (path "/0612bbdb-48b1-467f-9d3e-aa2a44e45a81"
-      (reference "TP12") (unit 1) (value "TestPoint") (footprint "TestPoint:TestPoint_Pad_2.5x2.5mm")
-    )
     (path "/88c93892-0d74-4376-bc39-1c17ac2d825d"

Commit message: v0.0 pcb checkin
Parts:
- added R10: 1k, Resistor_SMD:R_0805_2012Metric_Pad1.20x1.40mm_HandSolder, symbol Device:R
Connections:
- net at U3.25 (IO0): now also R10.1; no longer SW2.1
- new net: R10.2, SW2.1
Other:
- moved on the sheet: SW2
Changed lines of the file:
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@@
     (stroke (width 0) (type default) (color 0 0 0 0))
   )
-  (wire (pts (xy 180.975 89.535) (xy 180.975 90.805))
+  (wire (pts (xy 184.785 89.535) (xy 184.785 90.805))
     (stroke (width 0) (type default) (color 0 0 0 0))
   )
@@
     (stroke (width 0) (type default) (color 0 0 0 0))
   )
+  (wire (pts (xy 172.085 89.535) (xy 174.625 89.535))
+    (stroke (width 0) (type default) (color 0 0 0 0))
+  )
   (wire (pts (xy 128.905 101.6) (xy 128.905 106.045))
     (stroke (width 0) (type default) (color 0 0 0 0))
@@
     (stroke (width 0) (type default) (color 0 0 0 0))
   )
+  (wire (pts (xy 182.245 89.535) (xy 184.785 89.535))
+    (stroke (width 0) (type default) (color 0 0 0 0))
+  )
   (wire (pts (xy 190.5 112.395) (xy 189.23 112.395))
     (stroke (width 0) (type default) (color 0 0 0 0))
@@
     (stroke (width 0) (type default) (color 0 0 0 0))
   )
-  (wire (pts (xy 180.975 100.965) (xy 180.975 102.87))
+  (wire (pts (xy 184.785 100.965) (xy 184.785 102.87))
     (stroke (width 0) (type default) (color 0 0 0 0))
   )
@@
   )
   (wire (pts (xy 186.69 114.935) (xy 186.69 116.205))
-    (stroke (width 0) (type default) (color 0 0 0 0))
-  )
-  (wire (pts (xy 172.085 89.535) (xy 180.975 89.535))
     (stroke (width 0) (type default) (color 0 0 0 0))
   )
@@
     (pin "3")
   )
+  (symbol (lib_id "Device:R") (at 178.435 89.535 90) (unit 1)
+    (in_bom yes) (on_board yes) (fields_autoplaced)
+    (property "Reference" "R10" (id 0) (at 178.435 83.82 90))
+    (property "Value" "1k" (id 1) (at 178.435 86.36 90))
+    (property "Footprint" "Resistor_SMD:R_0805_2012Metric_Pad1.20x1.40mm_HandSolder" (id 2) (at 178.435 91.313 90)
+      (effects (font (size 1.27 1.27)) hide)
+    )
+    (property "Datasheet" "~" (id 3) (at 178.435 89.535 0)
+      (effects (font (size 1.27 1.27)) hide)
+    )
+    (pin "1")
+    (pin "2")
+  )
   (symbol (lib_id "power:GND") (at 186.69 125.095 0) (unit 1)
     (in_bom yes) (on_board yes) (fields_autoplaced)
@@
     (pin "1")
   )
-  (symbol (lib_id "Switch:SW_Push") (at 180.975 95.885 270) (unit 1)
+  (symbol (lib_id "Switch:SW_Push") (at 184.785 95.885 270) (unit 1)
     (in_bom yes) (on_board yes)
-    (property "Reference" "SW2" (id 0) (at 183.515 97.155 0)
-      (effects (font (size 1.27 1.27)) (justify left))
-    )
-    (property "Value" "FLASH" (id 1) (at 179.451 95.885 0))
-    (property "Footprint" "Button_Switch_THT:SW_PUSH-12mm_Wuerth-430476085716" (id 2) (at 186.055 95.885 0)
-      (effects (font (size 1.27 1.27)) hide)
-    )
-    (property "Datasheet" "~" (id 3) (at 186.055 95.885 0)
+    (property "Reference" "SW2" (id 0) (at 187.325 97.155 0)
+      (effects (font (size 1.27 1.27)) (justify left))
+    )
+    (property "Value" "FLASH" (id 1) (at 183.261 95.885 0))
+    (property "Footprint" "Button_Switch_THT:SW_PUSH-12mm_Wuerth-430476085716" (id 2) (at 189.865 95.885 0)
+      (effects (font (size 1.27 1.27)) hide)
+    )
+    (property "Datasheet" "~" (id 3) (at 189.865 95.885 0)
       (effects (font (size 1.27 1.27)) hide)
     )
@@
     (pin "1")
   )
-  (symbol (lib_id "power:GND") (at 180.975 102.87 0) (unit 1)
-    (in_bom yes) (on_board yes) (fields_autoplaced)
-    (property "Reference" "#PWR021" (id 0) (at 180.975 109.22 0)
-      (effects (font (size 1.27 1.27)) hide)
-    )
-    (property "Value" "GND" (id 1) (at 180.975 107.315 0))
-    (property "Footprint" "" (id 2) (at 180.975 102.87 0)
-      (effects (font (size 1.27 1.27)) hide)
-    )
-    (property "Datasheet" "" (id 3) (at 180.975 102.87 0)
+  (symbol (lib_id "power:GND") (at 184.785 102.87 0) (unit 1)
+    (in_bom yes) (on_board yes) (fields_autoplaced)
+    (property "Reference" "#PWR021" (id 0) (at 184.785 109.22 0)
+      (effects (font (size 1.27 1.27)) hide)
+    )
+    (property "Value" "GND" (id 1) (at 184.785 107.315 0))
+    (property "Footprint" "" (id 2) (at 184.785 102.87 0)
+      (effects (font (size 1.27 1.27)) hide)
+    )
+    (property "Datasheet" "" (id 3) (at 184.785 102.87 0)
       (effects (font (size 1.27 1.27)) hide)
     )
@@
       (reference "R9") (unit 1) (value "R_Photo") (footprint "OptoDevice:R_LDR_5.1x4.3mm_P3.4mm_Vertical")
     )
+    (path "/0245576c-3a10-420e-b216-e67a6904d6b5"
+      (reference "R10") (unit 1) (value "1k") (footprint "Resistor_SMD:R_0805_2012Metric_Pad1.20x1.40mm_HandSolder")
+    )
     (path "/53d21e73-5bfa-4153-b844-8c5b7eee3599"

Commit message: final versions I sent to TA, signing off for the week now
Parts:
- removed R7: 10k, Resistor_SMD:R_0805_2012Metric_Pad1.20x1.40mm_HandSolder, symbol Device:R
- removed U2: MAX14872ETC+, MAX14872ETC_:SON50P300X300X80-13N, symbol MAX14872ETC_:MAX14872ETC+
- added C15: 22u, Capacitor_SMD:C_0805_2012Metric_Pad1.18x1.45mm_HandSolder, symbol Device:C
- added U2: ZXBM5210-SP, Package_SO:Diodes_SO-8EP, symbol Driver_Motor:ZXBM5210-SP
Connections:
- net SNS is gone; now on net +9V: R1.1
- net +9V: now also U2.3 (VDD), U2.6 (VREF)
- net FWD: now also U2.4 (FWD)
- net GND: now also C15.2, U2.8 (GND), U2.9 (GND)
- net REV: now also U2.5 (REV)
- net at J3.1 (Pin_1): now also U2.7 (OUT2)
- net at J3.2 (Pin_2): now also U2.1 (OUT1)
- new net: C15.1, U2.2 (VM)
Other:
- moved on the sheet: C1, C12, C13, C14, C4, C8, J3, TP2, TP3

Commit message: final commit of the semester
Other:
- note added: "POWER MANAGEMENT"
- note removed: "POWER MANAGEMENT V1"
Changed lines of the file:
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@@
     (effects (font (size 3 3)) (justify left bottom))
   )
-  (text "POWER MANAGEMENT V1" (at 212.725 19.05 0)
+  (text "POWER MANAGEMENT" (at 215.646 18.288 0)
     (effects (font (size 3 3)) (justify left bottom))
   )
