File: kicad/v0.0/v0.0.kicad_pcb (KiCad board)
At the start: 2 copper layers, 53 parts, among them J1 USB_B_Micro, J2 9V_IN, J3 LED, J4 MOTOR, Q1 IRF520, SW1 RST, SW2 FLASH, SW3 OPEN/CLOSE, U1 MCP2221AxSL, U2 MAX14872ETC+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

Commit message: mbro isnt being such a bro
Parts:
- D1, D2: value D -> MBR0520; footprint Diode_SMD:D_SMA_Handsoldering -> Diode_SMD:D_SOD-123
- moved D1 51.6 mm to (175.0, 67.3)
- moved D2 45.8 mm to (134.4, 102.9), turned to 90 degrees
Connections:
- D1 pad 2: Net-(C10-Pad1) -> Net-(C3-Pad1)
- D2 pad 2: Net-(C3-Pad1) -> Net-(C10-Pad1)
Changed lines of the file:
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@@
     )
   )
-  (footprint "Diode_SMD:D_SMA_Handsoldering" (layer "F.Cu")
-    (at 134.874 99.822 90)
-    (descr "Diode SMA (DO-214AC) Handsoldering")
-    (tags "Diode SMA (DO-214AC) Handsoldering")
-    (property "Sheetfile" "v0.0.kicad_sch")
-    (property "Sheetname" "")
-    (attr smd)
-    (fp_text reference "D1" (at 0 2.482 90) (layer "F.SilkS")
-      (effects (font (size 1 1) (thickness 0.15)))
-    )
-    (fp_text value "D" (at 0 2.6 90) (layer "F.Fab")
-      (effects (font (size 1 1) (thickness 0.15)))
-    )
-    (fp_text user "${REFERENCE}" (at 0 -2.5 90) (layer "F.Fab")
-      (effects (font (size 1 1) (thickness 0.15)))
-    )
-    (fp_line (start -4.4 -1.65) (end -4.4 1.65) (layer "F.SilkS") (width 0.12))
-    (fp_line (start -4.4 1.65) (end 2.5 1.65) (layer "F.SilkS") (width 0.12))
-    (fp_line (start -4.4 -1.65) (end 2.5 -1.65) (layer "F.SilkS") (width 0.12))
-    (fp_line (start 4.5 -1.75) (end 4.5 1.75) (layer "F.CrtYd") (width 0.05))
-    (fp_line (start -4.5 1.75) (end -4.5 -1.75) (layer "F.CrtYd") (width 0.05))
-    (fp_line (start 4.5 1.75) (end -4.5 1.75) (layer "F.CrtYd") (width 0.05))
-    (fp_line (start -4.5 -1.75) (end 4.5 -1.75) (layer "F.CrtYd") (width 0.05))
-    (fp_line (start -0.64944 0.00102) (end 0.50118 0.75032) (layer "F.Fab") (width 0.1))
-    (fp_line (start -0.64944 0.00102) (end -1.55114 0.00102) (layer "F.Fab") (width 0.1))
-    (fp_line (start -2.3 1.5) (end -2.3 -1.5) (layer "F.Fab") (width 0.1))
-    (fp_line (start -0.64944 0.00102) (end 0.50118 -0.79908) (layer "F.Fab") (width 0.1))
-    (fp_line (start 2.3 -1.5) (end -2.3 -1.5) (layer "F.Fab") (width 0.1))
-    (fp_line (start 2.3 -1.5) (end 2.3 1.5) (layer "F.Fab") (width 0.1))
-    (fp_line (start 0.50118 0.00102) (end 1.4994 0.00102) (layer "F.Fab") (width 0.1))
-    (fp_line (start 2.3 1.5) (end -2.3 1.5) (layer "F.Fab") (width 0.1))
-    (fp_line (start -0.64944 -0.79908) (end -0.64944 0.80112) (layer "F.Fab") (width 0.1))
-    (fp_line (start 0.50118 0.75032) (end 0.50118 -0.79908) (layer "F.Fab") (width 0.1))
-    (pad "1" smd rect (at -2.5 0 90) (size 3.5 1.8) (layers "F.Cu" "F.Paste" "F.Mask")
+  (footprint "Diode_SMD:D_SOD-123" (layer "F.Cu")
+    (at 175.006 67.31 90)
+    (descr "SOD-123")
+    (tags "SOD-123")
+    (property "Sheetfile" "v0.0.kicad_sch")
+    (property "Sheetname" "")
+    (attr smd)
+    (fp_text reference "D1" (at 0 -2 90) (layer "F.SilkS")
+      (effects (font (size 1 1) (thickness 0.15)))
+    )
+    (fp_text value "MBR0520" (at 0 2.1 90) (layer "F.Fab")
+      (effects (font (size 1 1) (thickness 0.15)))
+    )
+    (fp_text user "${REFERENCE}" (at 0 -2 90) (layer "F.Fab")
+      (effects (font (size 1 1) (thickness 0.15)))
+    )
+    (fp_line (start -2.25 -1) (end 1.65 -1) (layer "F.SilkS") (width 0.12))
+    (fp_line (start -2.25 1) (end 1.65 1) (layer "F.SilkS") (width 0.12))
+    (fp_line (start -2.25 -1) (end -2.25 1) (layer "F.SilkS") (width 0.12))
+    (fp_line (start 2.35 -1.15) (end 2.35 1.15) (layer "F.CrtYd") (width 0.05))
+    (fp_line (start -2.35 -1.15) (end -2.35 1.15) (layer "F.CrtYd") (width 0.05))
+    (fp_line (start -2.35 -1.15) (end 2.35 -1.15) (layer "F.CrtYd") (width 0.05))
+    (fp_line (start 2.35 1.15) (end -2.35 1.15) (layer "F.CrtYd") (width 0.05))
+    (fp_line (start 0.25 0.4) (end -0.35 0) (layer "F.Fab") (width 0.1))
+    (fp_line (start -0.35 0) (end -0.35 -0.55) (layer "F.Fab") (width 0.1))
+    (fp_line (start -0.35 0) (end -0.35 0.55) (layer "F.Fab") (width 0.1))
+    (fp_line (start -0.75 0) (end -0.35 0) (layer "F.Fab") (width 0.1))
+    (fp_line (start 1.4 0.9) (end -1.4 0.9) (layer "F.Fab") (width 0.1))
+    (fp_line (start -1.4 0.9) (end -1.4 -0.9) (layer "F.Fab") (width 0.1))
+    (fp_line (start 1.4 -0.9) (end 1.4 0.9) (layer "F.Fab") (width 0.1))
+    (fp_line (start 0.25 0) (end 0.75 0) (layer "F.Fab") (width 0.1))
+    (fp_line (start 0.25 -0.4) (end 0.25 0.4) (layer "F.Fab") (width 0.1))
+    (fp_line (start -1.4 -0.9) (end 1.4 -0.9) (layer "F.Fab") (width 0.1))
+    (fp_line (start -0.35 0) (end 0.25 -0.4) (layer "F.Fab") (width 0.1))
+    (pad "1" smd rect (at -1.65 0 90) (size 0.9 1.2) (layers "F.Cu" "F.Paste" "F.Mask")
       (net 9 "+3V3") (pinfunction "K") (pintype "passive"))
-    (pad "2" smd rect (at 2.5 0 90) (size 3.5 1.8) (layers "F.Cu" "F.Paste" "F.Mask")
-      (net 10 "Net-(C10-Pad1)") (pinfunction "A") (pintype "passive"))
-    (model "${KICAD6_3DMODEL_DIR}/Diode_SMD.3dshapes/D_SMA.wrl"
+    (pad "2" smd rect (at 1.65 0 90) (size 0.9 1.2) (layers "F.Cu" "F.Paste" "F.Mask")
+      (net 1 "Net-(C3-Pad1)") (pinfunction "A") (pintype "passive"))
+    (model "${KICAD6_3DMODEL_DIR}/Diode_SMD.3dshapes/D_SOD-123.wrl"
       (offset (xyz 0 0 0))
       (scale (xyz 1 1 1))
@@
       (net 3 "+9V") (pinfunction "1") (pintype "passive"))
   )
-  (footprint "Diode_SMD:D_SMA_Handsoldering" (layer "F.Cu")
-    (at 168.16 71.96 180)
-    (descr "Diode SMA (DO-214AC) Handsoldering")
-    (tags "Diode SMA (DO-214AC) Handsoldering")
-    (property "Sheetfile" "v0.0.kicad_sch")
-    (property "Sheetname" "")
-    (attr smd)
-    (fp_text reference "D2" (at 0 2.41) (layer "F.SilkS")
-      (effects (font (size 1 1) (thickness 0.15)))
-    )
-    (fp_text value "D" (at 0 2.6) (layer "F.Fab")
-      (effects (font (size 1 1) (thickness 0.15)))
-    )
-    (fp_text user "${REFERENCE}" (at 0 -2.5) (layer "F.Fab")
-      (effects (font (size 1 1) (thickness 0.15)))
-    )
-    (fp_line (start -4.4 -1.65) (end -4.4 1.65) (layer "F.SilkS") (width 0.12))
-    (fp_line (start -4.4 1.65) (end 2.5 1.65) (layer "F.SilkS") (width 0.12))
-    (fp_line (start -4.4 -1.65) (end 2.5 -1.65) (layer "F.SilkS") (width 0.12))
-    (fp_line (start 4.5 -1.75) (end 4.5 1.75) (layer "F.CrtYd") (width 0.05))
-    (fp_line (start -4.5 -1.75) (end 4.5 -1.75) (layer "F.CrtYd") (width 0.05))
-    (fp_line (start 4.5 1.75) (end -4.5 1.75) (layer "F.CrtYd") (width 0.05))
-    (fp_line (start -4.5 1.75) (end -4.5 -1.75) (layer "F.CrtYd") (width 0.05))
-    (fp_line (start -2.3 1.5) (end -2.3 -1.5) (layer "F.Fab") (width 0.1))
-    (fp_line (start 2.3 -1.5) (end -2.3 -1.5) (layer "F.Fab") (width 0.1))
-    (fp_line (start 2.3 -1.5) (end 2.3 1.5) (layer "F.Fab") (width 0.1))
-    (fp_line (start 0.50118 0.75032) (end 0.50118 -0.79908) (layer "F.Fab") (width 0.1))
-    (fp_line (start 0.50118 0.00102) (end 1.4994 0.00102) (layer "F.Fab") (width 0.1))
-    (fp_line (start 2.3 1.5) (end -2.3 1.5) (layer "F.Fab") (width 0.1))
-    (fp_line (start -0.64944 0.00102) (end 0.50118 -0.79908) (layer "F.Fab") (width 0.1))
-    (fp_line (start -0.64944 -0.79908) (end -0.64944 0.80112) (layer "F.Fab") (width 0.1))
-    (fp_line (start -0.64944 0.00102) (end 0.50118 0.75032) (layer "F.Fab") (width 0.1))
-    (fp_line (start -0.64944 0.00102) (end -1.55114 0.00102) (layer "F.Fab") (width 0.1))
-    (pad "1" smd rect (at -2.5 0 180) (size 3.5 1.8) (layers "F.Cu" "F.Paste" "F.Mask")
+  (footprint "Diode_SMD:D_SOD-123" (layer "F.Cu")
+    (at 134.366 102.87 90)
+    (descr "SOD-123")
+    (tags "SOD-123")
+    (property "Sheetfile" "v0.0.kicad_sch")
+    (property "Sheetname" "")
+    (attr smd)
+    (fp_text reference "D2" (at 3.302 0 180) (layer "F.SilkS")
+      (effects (font (size 1 1) (thickness 0.15)))
+    )
+    (fp_text value "MBR0520" (at 0 2.1 90) (layer "F.Fab")
+      (effects (font (size 1 1) (thickness 0.15)))
+    )
+    (fp_text user "${REFERENCE}" (at 0 -2 90) (layer "F.Fab")
+      (effects (font (size 1 1) (thickness 0.15)))
+    )
+    (fp_line (start -2.25 -1) (end 1.65 -1) (layer "F.SilkS") (width 0.12))
+    (fp_line (start -2.25 1) (end 1.65 1) (layer "F.SilkS") (width 0.12))
+    (fp_line (start -2.25 -1) (end -2.25 1) (layer "F.SilkS") (width 0.12))
+    (fp_line (start -2.35 -1.15) (end -2.35 1.15) (layer "F.CrtYd") (width 0.05))
+    (fp_line (start 2.35 1.15) (end -2.35 1.15) (layer "F.CrtYd") (width 0.05))
+    (fp_line (start -2.35 -1.15) (end 2.35 -1.15) (layer "F.CrtYd") (width 0.05))
+    (fp_line (start 2.35 -1.15) (end 2.35 1.15) (layer "F.CrtYd") (width 0.05))
+    (fp_line (start 0.25 0.4) (end -0.35 0) (layer "F.Fab") (width 0.1))
+    (fp_line (start 1.4 -0.9) (end 1.4 0.9) (layer "F.Fab") (width 0.1))
+    (fp_line (start -1.4 -0.9) (end 1.4 -0.9) (layer "F.Fab") (width 0.1))
+    (fp_line (start -0.35 0) (end -0.35 0.55) (layer "F.Fab") (width 0.1))
+    (fp_line (start -0.75 0) (end -0.35 0) (layer "F.Fab") (width 0.1))
+    (fp_line (start -0.35 0) (end 0.25 -0.4) (layer "F.Fab") (width 0.1))
+    (fp_line (start -1.4 0.9) (end -1.4 -0.9) (layer "F.Fab") (width 0.1))
+    (fp_line (start 0.25 -0.4) (end 0.25 0.4) (layer "F.Fab") (width 0.1))
+    (fp_line (start 0.25 0) (end 0.75 0) (layer "F.Fab") (width 0.1))
+    (fp_line (start -0.35 0) (end -0.35 -0.55) (layer "F.Fab") (width 0.1))
+    (fp_line (start 1.4 0.9) (end -1.4 0.9) (layer "F.Fab") (width 0.1))
+    (pad "1" smd rect (at -1.65 0 90) (size 0.9 1.2) (layers "F.Cu" "F.Paste" "F.Mask")
       (net 9 "+3V3") (pinfunction "K") (pintype "passive"))
-    (pad "2" smd rect (at 2.5 0 180) (size 3.5 1.8) (layers "F.Cu" "F.Paste" "F.Mask")
-      (net 1 "Net-(C3-Pad1)") (pinfunction "A") (pintype "passive"))
-    (model "${KICAD6_3DMODEL_DIR}/Diode_SMD.3dshapes/D_SMA.wrl"
-      (offset (xyz 0 0 0))
-      (scale (xyz 1 1 1))
+    (pad "2" smd rect (at 1.65 0 90) (size 0.9 1.2) (layers "F.Cu" "F.Paste" "F.Mask")
+      (net 10 "Net-(C10-Pad1)") (pinfunction "A") (pintype "passive"))
+    (model "${KICAD6_3DMODEL_DIR}/Diode_SMD.3dshapes/D_SOD-123.wrl"
+      (offset (xyz 0 0 0))
+      (scale (xyz 1 1 1))

Commit message: general layout ready to be finalized
Parts:
- removed SW3: OPEN/CLOSE, Button_Switch_THT:SW_PUSH-12mm
- added J5: BUTTON, Connector_Molex:Molex_KK-254_AE-6410-02A_1x02_P2.54mm_Vertical, F.Cu at (163.6, 80.3)
- J3: value LED -> MOTOR
- J4: value MOTOR -> LED; footprint Connector_Molex:Molex_KK-254_AE-6410-02A_1x02_P2.54mm_Vertical -> Connector_Molex:Molex_KK-254_AE-6410-04A_1x04_P2.54mm_Vertical
- moved J3 82.3 mm to (124.7, 88.1), turned to 90 degrees
- moved TP3 79.8 mm to (146.2, 95.0)
- moved TP2 79.8 mm to (150.4, 95.0)
- moved C5 78.4 mm to (130.0, 92.7)
- moved Q1 74.0 mm to (138.2, 95.2)
- moved R5 73.6 mm to (135.1, 92.5), turned to 90 degrees
- moved TP1 73.0 mm to (133.1, 98.3)
- moved C14 71.3 mm to (147.7, 85.6)
- moved C13 70.7 mm to (137.4, 84.8)
- moved U2 61.7 mm to (132.1, 86.9)
- moved R7 58.0 mm to (133.4, 81.8), turned to 180 degrees
- moved R1 52.7 mm to (133.4, 78.2), turned to 180 degrees
- moved C8 52.6 mm to (128.8, 78.2), turned to 0 degrees
- moved C4 47.8 mm to (124.0, 81.8)
- moved C1 47.8 mm to (128.8, 81.8)
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Connections:
- J3 pad 1: Net-(J3-Pad1) -> Net-(U2-Pad11)
- J3 pad 2: GND -> Net-(U2-Pad2)
- J4 pad 1: Net-(J4-Pad1) -> GND
- J4 pad 2: Net-(J4-Pad2) -> Net-(R5-Pad2)
- R5 pad 2: Net-(J3-Pad1) -> Net-(R5-Pad2)
- U2 pad 11: Net-(J4-Pad2) -> Net-(U2-Pad11)
- U2 pad 2: Net-(J4-Pad1) -> Net-(U2-Pad2)
Routing:
- net +3V3: track 0.00 -> 52.1 mm, vias 0 -> 2
- net Net-(C6-Pad1): track 0.00 -> 25.2 mm
- net Net-(C3-Pad1): track 0.00 -> 17.0 mm
- net Net-(C7-Pad1): track 0.00 -> 16.8 mm
- net /V_PHOTO: track 0.00 -> 15.0 mm
- net Net-(J1-Pad3): track 0.00 -> 10.7 mm
- net GND: track 0.00 -> 10.7 mm
- net Net-(J1-Pad2): track 0.00 -> 10.4 mm
- net /RXD0: track 0.00 -> 9.78 mm
- net /TXD0: track 0.00 -> 9.48 mm
- net Net-(R2-Pad1): track 0.00 -> 8.71 mm
- net unconnected-(J1-Pad6): track 0.00 -> 8.63 mm
