File: kicad/v2.0/v2.0.kicad_pcb (KiCad board)
At the start: 2 copper layers, 54.1 x 99.1 mm, 34 parts, among them J1 9V_IN, J2 BUTTON, J3 LED STRIP, J4 MOTOR, J5 DEV BOARD LEFT, J6 DEV BOARD RIGHT, Q1 FQP30N06L, U1 L293D, U2 L7805

Commit message: minor changes to pcb
Parts:
- moved H1 69.2 mm to (124.2, 50.8)
- moved H2 69.2 mm to (124.2, 142.5)
- moved TP4 69.1 mm to (131.8, 51.6)
- moved C3 68.7 mm to (140.7, 132.1)
- moved J1 68.6 mm to (148.2, 131.0)
- moved TP3 68.6 mm to (158.0, 143.5)
- moved U2 68.6 mm to (157.2, 132.3)
- moved TP1 68.6 mm to (140.7, 143.3)
- moved TP2 68.6 mm to (140.7, 137.7)
- moved C2 68.6 mm to (154.7, 143.5)
- moved J3 68.6 mm to (132.8, 87.6)
- moved Q1 68.3 mm to (132.5, 79.8)
- moved R1 68.3 mm to (131.8, 95.2)
- moved TP7 68.3 mm to (131.8, 68.1)
- moved H4 67.9 mm to (172.5, 142.5)
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Routing:
- net +9V: track 123.1 -> 121.7 mm
- net +3V3: track 158.1 -> 159.4 mm
- net /LED: track 21.0 -> 22.0 mm
- net GND: vias 17 -> 29
Other:
- board size 54.1 x 99.1 mm -> 55.4 x 98.8 mm
- board text added: "Team 41 Smart Curtains V2.0 04/18/2023"
- board text removed: "Team 41 Smart Curtains V2.0 03/29/2023"

Commit message: final commit of the semester
Parts:
- moved C6 28.8 mm to (129.5, 94.7)
- moved C1 3.87 mm to (152.4, 115.8), turned to 180 degrees
- moved Q1 2.66 mm to (131.8, 77.2)
- moved TP7 2.59 mm to (131.3, 65.5)
- moved R2 2.29 mm to (166.6, 82.5)
- moved C4 2.27 mm to (152.4, 112.0), turned to 180 degrees
- moved C8 2.03 mm to (148.5, 106.2)
- moved TP5 2.03 mm to (165.4, 52.3)
- moved TP6 2.03 mm to (165.4, 57.4)
- moved U1 2.03 mm to (156.2, 103.9)
- moved R3 2.00 mm to (165.6, 62.0)
- moved R1 1.12 mm to (132.8, 94.7), turned to 90 degrees
- moved C7 1.05 mm to (152.4, 119.6), turned to 180 degrees
- moved TP8 1.02 mm to (165.4, 87.4)
- moved R4 1.02 mm to (167.3, 77.5)
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Routing:
- net +9V: track 121.7 -> 132.7 mm
- net /LED: track 22.0 -> 25.9 mm
- net /REV: track 63.4 -> 66.7 mm
- net Net-(J3-Pad2): track 11.6 -> 14.9 mm
- net /V_PHOTO: track 15.6 -> 18.2 mm
- net /FWD: track 56.3 -> 58.8 mm
- net Net-(J4-Pad6): track 43.6 -> 41.1 mm
- net Net-(J4-Pad5): track 30.9 -> 28.7 mm
- net Net-(J3-Pad1): track 7.65 -> 6.21 mm
- net Net-(R3-Pad1): track 18.7 -> 20.0 mm
- net +5V: track 78.3 -> 77.4 mm
- net GND: vias 29 -> 25
