File: kicad/v2.0/v2.0.kicad_sch (KiCad schematic)
At the start: 46 parts, among them J1 USB_B_Micro, J2 9V_IN, J3 MOTOR, J4 LED, J5 BUTTON, Q1 IRF520, SW1 RESET, SW2 FLASH, U1 MCP2221AxSL, U2 ZXBM5210-SP, U3 ESP32-WROOM-32, U4 AZ1117-3.3

Commit message: v2.0 is done
Parts:
- removed C11, C12, C13: 22u, Capacitor_SMD:C_0805_2012Metric_Pad1.18x1.45mm_HandSolder, symbol Device:C
- removed C2: .1u, Capacitor_SMD:C_0805_2012Metric_Pad1.18x1.45mm_HandSolder, symbol Device:C
- removed C3: .47u, Capacitor_SMD:C_0805_2012Metric_Pad1.18x1.45mm_HandSolder, symbol Device:C
- removed C7: 1u, Capacitor_SMD:C_0805_2012Metric_Pad1.18x1.45mm_HandSolder, symbol Device:C
- removed D1, D2: MBR0520, Diode_SMD:D_SOD-123, symbol Diode:MBR0520
- removed J1: USB_B_Micro, Connector_USB:USB_Micro-B_Molex-105133-0031, symbol Connector:USB_B_Micro
- removed J4: LED, Connector_Molex:Molex_KK-254_AE-6410-04A_1x04_P2.54mm_Vertical, symbol Connector:Conn_01x04_Male
- removed Q1: IRF520, IRF520:TO220BV, symbol IRF520:IRF520
- removed R3: 1k, Resistor_SMD:R_0805_2012Metric_Pad1.20x1.40mm_HandSolder, symbol Device:R
- removed R5: 10k, Resistor_SMD:R_0805_2012Metric_Pad1.20x1.40mm_HandSolder, symbol Device:R
- removed R6: 20k, Resistor_SMD:R_0805_2012Metric_Pad1.20x1.40mm_HandSolder, symbol Device:R
- removed R7: R_Photo, OptoDevice:R_LDR_5.1x4.3mm_P3.4mm_Vertical, symbol Device:R_Photo
- removed SW1: RESET, Button_Switch_THT:SW_PUSH_6mm, symbol Switch:SW_Push
- removed SW2: FLASH, Button_Switch_THT:SW_PUSH_6mm, symbol Switch:SW_Push
- removed TP1: LED, TestPoint:TestPoint_Pad_2.5x2.5mm, symbol Connector:TestPoint
- removed TP6: 5V, TestPoint:TestPoint_Pad_2.5x2.5mm, symbol Connector:TestPoint
- removed U1: MCP2221AxSL, Package_SO:SOIC-14_3.9x8.7mm_P1.27mm, symbol Interface_USB:MCP2221AxSL
- removed U2: ZXBM5210-SP, Package_SO:Diodes_SO-8EP, symbol Driver_Motor:ZXBM5210-SP
- removed U3: ESP32-WROOM-32, RF_Module:ESP32-WROOM-32, symbol RF_Module:ESP32-WROOM-32
- removed U4: AZ1117-3.3, Package_TO_SOT_SMD:SOT-89-3_Handsoldering, symbol Regulator_Linear:AZ1117-3.3
- added J3: LED STRIP, Connector_Molex:Molex_KK-254_AE-6410-02A_1x02_P2.54mm_Vertical, symbol Connector:Conn_01x02_Male
- added J5: DEV BOARD LEFT, Connector_PinSocket_2.54mm:PinSocket_1x19_P2.54mm_Vertical, symbol Connector:Conn_01x19_Female
- added J6: DEV BOARD RIGHT, Connector_PinSocket_2.54mm:PinSocket_1x19_P2.54mm_Vertical, symbol Connector:Conn_01x19_Female
- added Q1: FQP30N06L, Package_TO_SOT_THT:TO-220-3_Vertical, symbol Device:Q_NPN_BCE
- added R2: 3.3k, Resistor_SMD:R_0805_2012Metric_Pad1.20x1.40mm_HandSolder, symbol Device:R
- added R4: R_Photo, OptoDevice:R_LDR_5.1x4.3mm_P3.4mm_Vertical, symbol Device:R_Photo
- added TP4: 3V3, TestPoint:TestPoint_Pad_2.5x2.5mm, symbol Connector:TestPoint
- added TP7: LED, TestPoint:TestPoint_Pad_2.5x2.5mm, symbol Connector:TestPoint
- added TP8: V_PHOTO, TestPoint:TestPoint_Pad_2.5x2.5mm, symbol Connector:TestPoint
- added U1: L293D, Package_DIP:DIP-16_W7.62mm, symbol Driver_Motor:L293D
- added U2: L7805, Package_TO_SOT_THT:TO-220-3_Vertical, symbol Regulator_Linear:L7805
- C1: value .1u -> 0.1u
- C2: renamed from C10; value 22u -> 0.1u
- C3: renamed from C9; value 10u -> 0.33u
- R1: value 1k -> 100
- R3: renamed from R4; value 1k -> 10k
- TP3: renamed from TP5; value 3V3 -> 5V
- renumbered C8 to C7, C14 to C8, C15 to C9, J2 to J1, J5 to J2, J3 to J4, TP7 to TP1, TP4 to TP2, TP2 to TP5, TP3 to TP6
Connections:
- net GPIO34 is gone; now on net GND: J4.1 (Pin_1)
- net +9V: now also C6.1, R1.1, U1.8 (VCC2), U2.1 (IN); no longer C5.1
- net FWD: now also J6.11 (Pin_11), U1.2 (1A)
- net GND: now also C5.1, J5.14 (Pin_14), J6.12 (Pin_12), J6.19 (Pin_19), Q1.3 (E), R2.2, U1.12 (GND), U1.13 (GND), U1.4 (GND), U1.5 (GND), U2.2 (GND); no longer C5.2
- net LED: now also J5.15 (Pin_15), Q1.1 (B), TP7.1
- net REV: now also J6.10 (Pin_10), U1.7 (2A)
- net at R1.2: now also J3.1 (Pin_1)
- net at J4.5 (Pin_5): now also U1.6 (2Y)
- net at J4.6 (Pin_6): now also U1.3 (1Y)
- net at J2.1 (Pin_1), R3.1: now also J6.8 (Pin_8)
- net 3V3_INPUT renamed +5V
- net +5V: now also C5.2, J5.19 (Pin_19), U1.16 (VCC1), U2.3 (OUT); no longer J2.2 (Pin_2)
- net GPIO32 renamed ENCODER1
- net ENCODER1: now also J5.8 (Pin_8)
- net GPIO33 renamed +3V3
- net +3V3: now also J2.2 (Pin_2), J5.1 (Pin_1), R4.1, TP4.1, U1.1 (EN1,2)
- net GPIO35 renamed ENCODER2
- net ENCODER2: now also J5.7 (Pin_7)
- new net: J3.2 (Pin_2), Q1.2 (C)
- new net V_PHOTO: J6.7 (Pin_7), R2.1, R4.2, TP8.1
Other:
- note added: "DEV BOARD"
- note added: "LED & PHOTO_READ"
- note added: "POWER MANAGEMENT"
- note removed: "CONTROL UNIT"
- note removed: "LED"
- note removed: "POWER MANAGEMENT V1"
- note removed: "USB to UART"
- note removed: "used to flash the board NO TOUCHY"
- moved on the sheet: C1, C4, C7, C8, C9, J2, J4, R3, TP5, TP6
